Commit message: shaft cannot turning around and around, but others works fine

File: src/motorsim_description/urdf/stepmotor.xacro (robot description, xacro)
@@ -19,6 +19,6 @@
         ixy="0"
         ixz="0"
-        iyy="0"
-        iyz="-1"
+        iyy="1"
+        iyz="0"
         izz="1" />
     </inertial>
@@ -51,15 +51,15 @@
     <inertial>
       <origin
-        xyz="-0.000861121867187112 -0.000341800191336777 1.53512652504286E-05"
+        xyz="-0.00012249817140968 0.0141141740469127 2.16712378782197E-10"
         rpy="0 0 0" />
       <mass
-        value="0.5" />
+        value="0.005" />
       <inertia
-        ixx="1"
+        ixx="0.1"
         ixy="0"
         ixz="0"
-        iyy="1"
+        iyy="0.0001"
         iyz="0"
-        izz="1" />
+        izz="0.0001" />
     </inertial>
     <visual>
@@ -89,8 +89,8 @@
   <joint
     name="motorjoint"
-    type="revolute">
+    type="continuous">
     <origin
-      xyz="0 0 0"
-      rpy="0 0 0" />
+      xyz="-0.0008591 -0.0003418 0"
+      rpy="1.5708 0 0" />
     <parent
       link="motorbase" />
@@ -98,6 +98,6 @@
       link="shaft" />
     <axis
-      xyz="0 0 1" />
-<limit upper="3000" lower="-3000" effort="3000" velocity="1000"/>
+      xyz="0 1 0" />
+<limit upper="360" lower="-360" effort="100" velocity="100"/>
   </joint>
 </robot>

Commit message: Still not spinning

File: src/motorsim_description/urdf/stepmotor.xacro (robot description, xacro)
@@ -7,5 +7,5 @@
     </plugin>
   </gazebo>
-  <!-- Used for fixing robot to Gazebo 'base_link' -->
+  <!-- Used for fixing robot to Gazebo 'base_link'-->
   <link name="world"/>
   <joint name="fixed" type="fixed">
@@ -16,15 +16,15 @@
     <inertial>
       <origin
-        xyz="-1.73472347597681E-18 -0.000239932345629558 0.0193535938441835"
+        xyz="-1.73472347597681E-18 -0.000240520210148032 0.01935323513063"
         rpy="0 0 0" />
       <mass
-        value="0.522970509231659" />
+        value="0.521692297282674" />
       <inertia
-        ixx="0.000143448111633865"
-        ixy="3.62654681759611E-22"
-        ixz="-2.1703853094235E-14"
-        iyy="0.000140708440567143"
-        iyz="-1.73806186578438E-06"
-        izz="0.000150994356797971" />
+        ixx="0.000143281413851519"
+        ixy="5.0594989079774E-23"
+        ixz="-2.17038531015825E-14"
+        iyy="0.000140541816548591"
+        iyz="-1.73801685528978E-06"
+        izz="0.000150985116656737" />
     </inertial>
     <visual>
@@ -56,5 +56,5 @@
     <inertial>
       <origin
-        xyz="-5.57804855252468E-05 3.64428279169271E-05 0.0316447657775446"
+        xyz="-5.57804855252433E-05 3.6442827916934E-05 -0.0323552342224554"
         rpy="0 0 0" />
       <mass
@@ -93,8 +93,8 @@
   </link>
   <joint
-    name="motorjoint"
+    name="joint1"
     type="continuous">
     <origin
-      xyz="0 0 0"
+      xyz="0 0 0.064"
       rpy="0 0 0" />
     <parent
@@ -107,5 +107,5 @@
   <transmission name="tran1">
     <type>transmission_interface/SimpleTransmission</type>
-    <joint name="motorjoint">
+    <joint name="joint1">
       <hardwareInterface>hardware_interface/VelocityJointInterface</hardwareInterface>
     </joint>
